File: DoAnSpring2013/analog-out-and-pwr-amp.brd (EAGLE design)
At the start: 100 x 80 mm, 25 parts, among them IC1 TL082, U1 TEA2025B

Commit message: minor changes
Parts:
- added JP5: (no value), datle-conn:1X01
- moved C13 8.63 mm to (74.0, 18.1), turned to 0 degrees
Connections:
- net GND: now also JP5.1
Routing:
- net GND: track 204.2 -> 199.0 mm
- net N$13: track 24.2 -> 27.3 mm
