File: DoAnSpring2013/analog-out-and-pwr-amp.sch (EAGLE design)
At the start: 25 parts, among them IC1 TL082, U1 TEA2025B

Commit message: minor changes
Parts:
- added JP5: (no value), datle-conn:PINHD-1X1
Connections:
- net GND: now also JP5.1
Changed lines of the file:
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@@
 <part name="JP3" library="datle-conn" deviceset="PINHD-1X1" device=""/>
 <part name="JP4" library="datle-conn" deviceset="PINHD-1X2" device="0.5&quot;" value="SPEAKER"/>
+<part name="JP5" library="datle-conn" deviceset="PINHD-1X1" device=""/>
+<part name="GND11" library="supply1" deviceset="GND" device=""/>
 </parts>
 <sheets>
@@
 <instance part="JP3" gate="G$1" x="171.45" y="62.23" rot="R90"/>
 <instance part="JP4" gate="G$1" x="166.37" y="-8.89"/>
+<instance part="JP5" gate="G$1" x="189.23" y="62.23" rot="R90"/>
+<instance part="GND11" gate="1" x="189.23" y="49.53"/>
 </instances>
 <busses>
@@
 <wire x1="176.53" y1="15.24" x2="176.53" y2="16.51" width="0.1524" layer="91"/>
 </segment>
+<segment>
+<pinref part="JP5" gate="G$1" pin="1"/>
+<pinref part="GND11" gate="1" pin="GND"/>
+<wire x1="189.23" y1="59.69" x2="189.23" y2="52.07" width="0.1524" layer="91"/>
+</segment>
 </net>
