File: DoAnSpring2013/mmcaudio-analog-in.brd (EAGLE design)
At the start: 100 x 80 mm, 24 parts, among them IC1 TL082, IC2 TL082

Commit message: minor changes
Routing:
- net N$9: track 19.7 -> 21.0 mm
Changed lines of the file:
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@@
 <grid distance="6.25" unitdist="mil" unit="mil" style="lines" multiple="1" display="yes" altdistance="0.025" altunitdist="inch" altunit="inch"/>
 <layers>
-<layer number="1" name="Top" color="4" fill="1" visible="yes" active="yes"/>
+<layer number="1" name="Top" color="4" fill="1" visible="no" active="yes"/>
 <layer number="16" name="Bottom" color="1" fill="1" visible="yes" active="yes"/>
 <layer number="17" name="Pads" color="2" fill="1" visible="yes" active="yes"/>
 <layer number="18" name="Vias" color="2" fill="1" visible="yes" active="yes"/>
-<layer number="19" name="Unrouted" color="6" fill="1" visible="yes" active="yes"/>
-<layer number="20" name="Dimension" color="15" fill="1" visible="yes" active="yes"/>
-<layer number="21" name="tPlace" color="7" fill="1" visible="yes" active="yes"/>
-<layer number="22" name="bPlace" color="7" fill="1" visible="yes" active="yes"/>
-<layer number="23" name="tOrigins" color="15" fill="1" visible="yes" active="yes"/>
-<layer number="24" name="bOrigins" color="15" fill="1" visible="yes" active="yes"/>
-<layer number="25" name="tNames" color="7" fill="1" visible="yes" active="yes"/>
-<layer number="26" name="bNames" color="7" fill="1" visible="yes" active="yes"/>
-<layer number="27" name="tValues" color="7" fill="1" visible="yes" active="yes"/>
-<layer number="28" name="bValues" color="7" fill="1" visible="yes" active="yes"/>
+<layer number="19" name="Unrouted" color="6" fill="1" visible="no" active="yes"/>
+<layer number="20" name="Dimension" color="15" fill="1" visible="no" active="yes"/>
+<layer number="21" name="tPlace" color="7" fill="1" visible="no" active="yes"/>
+<layer number="22" name="bPlace" color="7" fill="1" visible="no" active="yes"/>
+<layer number="23" name="tOrigins" color="15" fill="1" visible="no" active="yes"/>
+<layer number="24" name="bOrigins" color="15" fill="1" visible="no" active="yes"/>
+<layer number="25" name="tNames" color="7" fill="1" visible="no" active="yes"/>
+<layer number="26" name="bNames" color="7" fill="1" visible="no" active="yes"/>
+<layer number="27" name="tValues" color="7" fill="1" visible="no" active="yes"/>
+<layer number="28" name="bValues" color="7" fill="1" visible="no" active="yes"/>
 <layer number="29" name="tStop" color="7" fill="3" visible="no" active="yes"/>
 <layer number="30" name="bStop" color="7" fill="6" visible="no" active="yes"/>
@@
 <contactref element="C6" pad="-"/>
 <wire x1="47.01" y1="10.16" x2="45.4025" y2="10.16" width="0.3048" layer="16"/>
-<wire x1="45.4025" y1="10.16" x2="44.1325" y2="11.43" width="0.3048" layer="16"/>
+<wire x1="45.4025" y1="10.16" x2="44.529375" y2="11.033125" width="0.3048" layer="16"/>
+<wire x1="44.529375" y1="11.033125" x2="44.1325" y2="11.43" width="0.3048" layer="16"/>
 <wire x1="44.1325" y1="11.43" x2="41.91" y2="11.43" width="0.3048" layer="16"/>
 <wire x1="43.18" y1="24.13" x2="43.18" y2="21.59" width="0.3048" layer="16"/>
-<wire x1="43.18" y1="21.59" x2="43.4975" y2="21.59" width="0.3048" layer="16"/>
-<wire x1="43.4975" y1="21.59" x2="45.085" y2="20.0025" width="0.3048" layer="16"/>
-<wire x1="45.085" y1="20.0025" x2="45.085" y2="12.3825" width="0.3048" layer="16"/>
-<wire x1="45.085" y1="12.3825" x2="44.1325" y2="11.43" width="0.3048" layer="16"/>
+<wire x1="43.4975" y1="21.59" x2="44.29125" y2="21.59" width="0.3048" layer="16"/>
+<wire x1="44.29125" y1="21.59" x2="46.19625" y2="19.685" width="0.3048" layer="16"/>
+<wire x1="46.19625" y1="19.685" x2="46.19625" y2="12.7" width="0.3048" layer="16"/>
+<wire x1="46.19625" y1="12.7" x2="44.529375" y2="11.033125" width="0.3048" layer="16"/>
+<wire x1="43.4975" y1="21.59" x2="43.18" y2="21.59" width="0" layer="19" extent="16-16"/>
 </signal>
 <signal name="N$10">

Commit message: begin routing main board
Parts:
- added C10, C13: 222, datle-discrete:C025-060X050
- added C11, C12, C15, C18, C7, C9: 100uF, datle-discrete:POL-CAP-COMMON
- added C14, C8: 223, datle-discrete:C025-060X050
- added C16, C19: 104, datle-discrete:C025-060X050
- added C17: (no value), datle-discrete:POL-CAP-COMMON
- added IC3: TL082, datle-analogic:DIP08
- added JP10, JP7, JP9: (no value), datle-conn:1X01
- added JP6: (no value), pinhead:1X04
- added JP8: SPEAKER, datle-conn:1X02/0.5"
- added R11: 6.8k, datle-discrete:R-US-COMMON
- added R12: 27k, datle-discrete:R-US-COMMON
- added R13, R14: 1.5k, datle-discrete:R-US-COMMON
- added R15: 10k, datle-discrete:RTRIM-COMMON
- added R16: 10k, datle-discrete:R-US-COMMON
- added U1: TEA2025B, datle-analogic:DIP254P762X510-16
Connections:
- new net N$14: C8.1, R11.2, R12.1
- new net N$15: C10.2, IC3.3, R12.2
- new net N$16: C8.2, IC3.1, IC3.2, R13.1
- new net N$17: C14.1, R13.2, R14.2
- new net N$18: C13.2, IC3.6, R14.1
- new net N$19: C14.2, C17.+, IC3.5, IC3.7
- new net N$20: JP7.1, R11.1
- new net N$21: C17.-, JP9.1, R15.3
- new net N$22: C9.+, U1.11
- new net N$23: C11.+, U1.6
- new net N$24: C11.-, U1.1
- new net N$25: C18.-, C19.2, JP8.1, U1.15
- new net N$26: C18.+, U1.14
- new net N$27: C15.-, C16.2, JP8.2, U1.2
- new net N$28: C15.+, U1.3
- new net N$29: C12.+, U1.8
- new net N$30: R15.1, R16.1
- new net PWR_AMP: R15.2, U1.10
- net +12V: now also C7.+, IC3.4, JP6.3, U1.16
- net -12V: now also IC3.8, JP6.2
- net GND: now also C10.1, C12.-, C13.1, C16.1, C19.1, C7.-, C9.-, JP10.1, JP6.1, R16.2, U1.12, U1.13, U1.4, U1.5, U1.7, U1.9
- net VCC: now also JP6.4
