File: DoAnSpring2013/mmcaudio.brd (EAGLE design)
At the start: 172.7 x 111.4 mm, 83 parts, among them IC1 TL082, IC2 TL082, IC3 LM1117, IC4 TL082, IC5 TL082, U1 DAC0808LCN, U2 TEA2025B, X1 HD44780LCD-1602

Commit message: add button B1 & B2
Parts:
- removed R31: 10k, datle-discrete:POT
- added R3: 1k, datle-discrete:R-US-COMMON
- added S2, S3: (no value), datle-switch:B3F-10XX
- C14, C15: value 223 -> 22p
- C16: value 223 -> 104
- R11: value 10k -> 1k
- R12: value 1k -> 330
- R13: value 330 -> 10k
- R14: value 10k -> 330
- R15: value 330 -> 100
- R16: value 100 -> 6.8k
- R22: value 6.8k -> 2k2
- R23: value 2k2 -> 5k
- R24: value 5k -> 2k2
- R25: value 2k2 -> 6.8k
- R26, R6: value 6.8k -> 27k
- R27: value 27k -> 1.5k
- R29: value 1.5k -> 10k
- R30: device datle-discrete:R-US-COMMON -> datle-discrete:POT
- R4: value 1k -> 100k; device datle-discrete:R-US-COMMON -> datle-discrete:RTRIM-COMMON
- R5: value 100k -> 6.8k; device datle-discrete:RTRIM-COMMON -> datle-discrete:R-US-COMMON
- R7: value 27k -> 3.3k
- R9: value 3.3k -> 10k
- moved Q1 184.5 mm to (78.7, 63.5), flipped to the bottom, turned to 270 degrees
- moved D1 180.5 mm to (63.5, 94.0), turned to 270 degrees
- moved C4 161.5 mm to (41.9, 105.4), turned to 270 degrees
- moved C7 156.2 mm to (53.3, 82.5), turned to 90 degrees
- moved C3 151.4 mm to (38.1, 105.4), turned to 270 degrees
- moved R11 144.8 mm to (58.4, 95.2), turned to 270 degrees
- moved R6 141.7 mm to (29.2, 108.0), turned to 180 degrees
- moved R12 141.1 mm to (8.89, 33.0)
- moved C15 130.8 mm to (78.7, 54.6), turned to 180 degrees
- moved R10 128.8 mm to (54.6, 95.2), turned to 90 degrees
- moved C14 118.9 mm to (78.7, 71.1), turned to 180 degrees
- moved R9 112.9 mm to (50.8, 95.2), turned to 90 degrees
- moved R4 111.5 mm to (11.4, 106.7), turned to 270 degrees
- moved S1 101.4 mm to (-119.4, -2.54)
- moved C2 98.4 mm to (19.1, 83.8)
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Connections:
- net ADC: now also R11.1; no longer R12.1
- net B1: now also S1.1, S1.2
- net B2: now also S2.1, S2.2
- net CLK: now also R20.2, R21.1; no longer R21.2, R22.1
- net CONTR: now also R14.1; no longer R15.1
- net CS: now also R16.2, R17.1; no longer R17.2, R18.1
- net GND: now also R10.2, R12.1, R16.1, R18.1, R20.1, R23.1, R30.3, S2.3, S2.4, S3.3, S3.4; no longer R11.2, R13.1, R17.1, R19.1, R21.1, R24.1, R31.3
- net IOUT: now also R24.1; no longer R26.1
- net MOSI: now also R18.2, R19.1; no longer R19.2, R20.1
- net N$10: now also R9.1; no longer R11.1
- net N$11: now also R11.2; no longer R12.2
- net N$14: now also R25.2, R26.1; no longer R26.2, R27.1
- net N$15: now also R26.2; no longer R27.2
- net N$16: now also R27.1; no longer R28.1
- net N$17: now also R27.2; no longer R29.2
- net N$18: now also R28.1; no longer R29.1
- net N$2: now also R3.2, R4.1; no longer R4.2, R5.1
- net N$21: now also R29.1; no longer R30.1
- net N$3: now also R4.2, R5.1; no longer R5.2, R6.1
- net N$30: now also R29.2, R30.1; no longer R30.2, R31.1
- net N$31: now also R3.1; no longer R4.1
- net N$32: now also R15.1; no longer R16.1
- net N$34: now also R24.2; no longer R25.2
- net N$36: now also R17.2; no longer R18.2
- net N$37: now also R12.2; no longer R13.2
- net N$38: now also R19.2; no longer R20.2
- net N$4: now also R5.2, R6.1; no longer R6.2, R7.1
- net N$40: now also R21.2; no longer R22.2
- net N$5: now also R6.2; no longer R7.2
- net N$6: now also R7.1; no longer R8.1
- net N$7: now also R7.2; no longer R9.2
- net N$8: now also R8.1; no longer R9.1
- net PWR_AMP: now also R30.2; no longer R31.2
- net RESET: now also R13.1, S3.1, S3.2; no longer R14.1, S1.1, S1.2
- net VCC: now also R13.2, R15.2, R22.2, R9.2; no longer R10.2, R14.2, R16.2, R23.2
- net VDD: now also R14.2; no longer R15.2
- net VREF+: now also R22.1; no longer R23.1
- net VREF-: now also R23.2; no longer R24.2

Commit message: routing failed 12:56SA 20131105
Parts:
- removed JP7: SPEAKER, datle-conn:1X02/0.5"
- removed JP8: (no value), datle-conn:1X01
- JP5: value (none) -> SPEAKER; device datle-conn:1X06 -> datle-conn:1X02/0.5"
- JP6: device datle-conn:JP1 -> datle-conn:1X01
- R14: value 330 -> 4k7
- moved R29 269.5 mm to (158.8, 48.3), turned to 270 degrees
- moved JP6 265.9 mm to (248.6, 91.1)
- moved JP3 260.3 mm to (215.6, 134.3)
- moved C30 254.7 mm to (142.2, 57.1), turned to 270 degrees
- moved R28 254.0 mm to (154.9, 48.3), turned to 270 degrees
- moved R30 250.3 mm to (157.5, 66.0)
- moved JP2 249.5 mm to (201.0, 110.5)
- moved C25 241.6 mm to (149.9, 96.5), turned to 90 degrees
- moved R27 238.7 mm to (151.1, 48.3), turned to 270 degrees
- moved R22 237.4 mm to (118.1, 61.0), turned to 270 degrees
- moved C29 236.2 mm to (147.3, 39.4), turned to 180 degrees
- moved R15 235.8 mm to (110.5, 39.4), turned to 180 degrees
- moved R14 229.6 mm to (94.0, 29.2), turned to 180 degrees
- moved C28 224.1 mm to (141.0, 39.4)
- moved U2 216.5 mm to (135.9, 82.5)
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Connections:
- removed net N$42: JP5.2, JP6.1
- net D4: now also U$1.38; no longer U$1.35
- net D5: now also U$1.37; no longer U$1.36
- net D6: now also U$1.36; no longer U$1.37
- net D7: now also U$1.35; no longer U$1.38
- net GND: now also JP5.2; no longer JP5.3, JP7.2
- net N$21: now also JP6.1; no longer JP8.1
- net N$25: now also JP5.1; no longer JP7.1
- net PGC: no longer JP5.5
- net PGD: no longer JP5.4
- net RESET: no longer JP5.1
- net VCC: no longer JP6.2
Routing:
- net GND: track 0.00 -> 976.0 mm, vias 0 -> 2
- net +12V: track 0.00 -> 428.9 mm
- net VCC: track 0.00 -> 213.6 mm
- net -12V: track 0.00 -> 177.9 mm
- net D4: track 0.00 -> 175.6 mm
- net D5: track 0.00 -> 167.6 mm
- net D6: track 0.00 -> 159.4 mm
- net D7: track 0.00 -> 152.4 mm
- net RS: track 0.00 -> 110.3 mm, vias 0 -> 2
- net E: track 0.00 -> 109.9 mm, vias 0 -> 2
- net N$9: track 0.00 -> 86.3 mm
- net MISO: track 0.00 -> 79.6 mm
- net N$15: track 0.00 -> 73.9 mm
- net +3V3: track 0.00 -> 44.8 mm
- net N$40: track 0.00 -> 44.6 mm, vias 0 -> 2
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Other:
- board size 172.7 x 111.4 mm -> 173 x 114.3 mm

Commit message: failed 3:02 20131105
Routing:
- net A5: track 0.00 -> 40.4 mm
- net VCC: track 213.6 -> 250.3 mm, vias 0 -> 2
- net N$40: track 44.6 -> 39.5 mm
- net RS: track 110.3 -> 112.7 mm
- net A6: track 39.7 -> 38.2 mm
- net A7: track 42.9 -> 41.7 mm
- net E: track 109.9 -> 110.7 mm
Changed lines of the file:
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@@
 <wire x1="34.4986" y1="32.7914" x2="35.56" y2="31.73" width="0.8128" layer="1"/>
 <wire x1="73.66" y1="69.85" x2="71.4375" y2="69.85" width="0.6096" layer="1"/>
-<wire x1="71.4375" y1="69.85" x2="35.56" y2="69.85" width="0.6096" layer="1"/>
+<wire x1="71.4375" y1="69.85" x2="40.3225" y2="69.85" width="0.6096" layer="1"/>
+<wire x1="40.3225" y1="69.85" x2="35.56" y2="69.85" width="0.6096" layer="1"/>
 <wire x1="35.56" y1="69.85" x2="33.02" y2="72.39" width="0.6096" layer="1"/>
 <wire x1="118.11" y1="55.88" x2="116.205" y2="55.88" width="0.4064" layer="1"/>
@@
 <wire x1="105.41" y1="39.37" x2="107.315" y2="39.37" width="0.3048" layer="1"/>
 <wire x1="107.315" y1="39.37" x2="110.1725" y2="42.2275" width="0.3048" layer="1"/>
-<wire x1="110.1725" y1="42.2275" x2="110.1725" y2="56.8325" width="0.3048" layer="1"/>
 <wire x1="110.1725" y1="56.8325" x2="109.855" y2="57.15" width="0.3048" layer="1"/>
-<wire x1="33.02" y1="72.39" x2="50.8" y2="100.33" width="0" layer="19" extent="1-1"/>
+<wire x1="50.8" y1="100.33" x2="50.4825" y2="100.33" width="0.4064" layer="1"/>
+<wire x1="50.4825" y1="100.33" x2="48.5775" y2="98.425" width="0.4064" layer="1"/>
+<via x="48.5775" y="98.425" extent="1-16" drill="0.6" shape="square"/>
+<wire x1="48.5775" y1="98.425" x2="48.5775" y2="76.5175" width="0.4064" layer="16"/>
+<via x="48.5775" y="76.5175" extent="1-16" drill="0.6" shape="square"/>
+<wire x1="48.5775" y1="76.5175" x2="46.99" y2="76.5175" width="0.4064" layer="1"/>
+<wire x1="46.99" y1="76.5175" x2="40.3225" y2="69.85" width="0.4064" layer="1"/>
+<wire x1="110.1725" y1="56.8325" x2="111.125" y2="55.88" width="0.4064" layer="1"/>
+<wire x1="111.125" y1="55.88" x2="111.125" y2="43.18" width="0.4064" layer="1"/>
+<wire x1="111.125" y1="43.18" x2="110.1725" y2="42.2275" width="0.4064" layer="1"/>
+<wire x1="88.9" y1="74.93" x2="107.95" y2="57.15" width="0" layer="19" extent="1-1"/>
 <wire x1="35.56" y1="31.73" x2="33.04" y2="16.51" width="0" layer="19" extent="1-1"/>
-<wire x1="107.95" y1="57.15" x2="88.9" y2="74.93" width="0" layer="19" extent="1-1"/>
 </signal>
 <signal name="ADC">
@@
 <wire x1="96.9" y1="34.73" x2="96.9" y2="36.7675" width="0.4064" layer="1"/>
 <wire x1="96.9" y1="36.7675" x2="96.2025" y2="37.465" width="0.4064" layer="1"/>
-<wire x1="96.2025" y1="37.465" x2="53.975" y2="37.465" width="0.4064" layer="1"/>
-<wire x1="53.975" y1="37.465" x2="48.5775" y2="42.8625" width="0.4064" layer="1"/>
-<wire x1="48.5775" y1="42.8625" x2="48.5775" y2="45.4025" width="0.4064" layer="1"/>
-<via x="48.5775" y="45.4025" extent="1-16" drill="0.6" diameter="1.4224" shape="square"/>
-<wire x1="48.5775" y1="45.4025" x2="48.5775" y2="73.66" width="0.4064" layer="16"/>
+<wire x1="96.2025" y1="37.465" x2="50.165" y2="37.465" width="0.4064" layer="1"/>
+<via x="48.26" y="39.37" extent="1-16" drill="0.6" diameter="1.4224" shape="square"/>
+<wire x1="48.26" y1="39.37" x2="48.5775" y2="73.66" width="0.4064" layer="16"/>
 <via x="48.5775" y="73.66" extent="1-16" drill="0.6" diameter="1.4224" shape="square"/>
 <wire x1="48.5775" y1="73.66" x2="67.6275" y2="73.66" width="0.4064" layer="1"/>
 <wire x1="67.6275" y1="73.66" x2="71.4375" y2="77.47" width="0.4064" layer="1"/>
 <wire x1="71.4375" y1="77.47" x2="73.66" y2="77.47" width="0.4064" layer="1"/>
+<wire x1="50.165" y1="37.465" x2="48.26" y2="39.37" width="0.4064" layer="1"/>
 </signal>
 <signal name="E">
@@
 <wire x1="101.98" y1="34.73" x2="101.98" y2="37.72" width="0.4064" layer="1"/>
 <wire x1="101.98" y1="37.72" x2="100.965" y2="38.735" width="0.4064" layer="1"/>
-<wire x1="100.965" y1="38.735" x2="54.2925" y2="38.735" width="0.4064" layer="1"/>
-<wire x1="54.2925" y1="38.735" x2="50.8" y2="42.2275" width="0.4064" layer="1"/>
-<wire x1="50.8" y1="42.2275" x2="50.8" y2="46.99" width="0.4064" layer="1"/>
-<via x="50.8" y="46.99" extent="1-16" drill="0.6" diameter="1.4224" shape="square"/>
-<wire x1="50.8" y1="46.99" x2="50.8" y2="72.0725" width="0.4064" layer="16"/>
+<wire x1="100.965" y1="38.735" x2="53.0225" y2="38.735" width="0.4064" layer="1"/>
+<via x="50.8" y="40.9575" extent="1-16" drill="0.6" diameter="1.4224" shape="square"/>
+<wire x1="50.8" y1="40.9575" x2="50.8" y2="72.0725" width="0.4064" layer="16"/>
 <via x="50.8" y="72.0725" extent="1-16" drill="0.6" diameter="1.4224" shape="square"/>
 <wire x1="50.8" y1="72.0725" x2="68.8975" y2="72.0725" width="0.4064" layer="1"/>
 <wire x1="68.8975" y1="72.0725" x2="71.755" y2="74.93" width="0.4064" layer="1"/>
 <wire x1="71.755" y1="74.93" x2="73.66" y2="74.93" width="0.4064" layer="1"/>
+<wire x1="53.0225" y1="38.735" x2="50.8" y2="40.9575" width="0.4064" layer="1"/>
 </signal>
 <signal name="PGD">
@@
 <contactref element="U$1" pad="22"/>
 <contactref element="U1" pad="8"/>
-<wire x1="88.9" y1="49.53" x2="95.5675" y2="49.53" width="0.3048" layer="1"/>
-<wire x1="95.5675" y1="49.53" x2="98.1075" y2="46.99" width="0.3048" layer="1"/>
 <wire x1="98.1075" y1="46.99" x2="100.33" y2="46.99" width="0.3048" layer="1"/>
+<wire x1="88.9" y1="49.53" x2="92.075" y2="49.53" width="0.4064" layer="1"/>
+<wire x1="92.075" y1="49.53" x2="94.615" y2="46.99" width="0.4064" layer="1"/>
+<wire x1="94.615" y1="46.99" x2="98.1075" y2="46.99" width="0.4064" layer="1"/>
 </signal>
 <signal name="A5">
 <contactref element="U$1" pad="21"/>
 <contactref element="U1" pad="9"/>
-<wire x1="88.9" y1="46.99" x2="107.95" y2="46.99" width="0" layer="19" extent="1-1"/>
+<wire x1="88.9" y1="46.99" x2="88.265" y2="46.99" width="0.4064" layer="1"/>
+<wire x1="88.265" y1="46.99" x2="86.36" y2="48.895" width="0.4064" layer="1"/>
+<wire x1="86.36" y1="48.895" x2="86.36" y2="50.165" width="0.4064" layer="1"/>
+<wire x1="86.36" y1="50.165" x2="86.995" y2="50.8" width="0.4064" layer="1"/>
+<wire x1="86.995" y1="50.8" x2="92.3925" y2="50.8" width="0.4064" layer="1"/>
+<wire x1="92.3925" y1="50.8" x2="94.9325" y2="48.26" width="0.4064" layer="1"/>
+<wire x1="94.9325" y1="48.26" x2="102.235" y2="48.26" width="0.4064" layer="1"/>
+<wire x1="102.235" y1="48.26" x2="103.8225" y2="49.8475" width="0.4064" layer="1"/>
+<wire x1="103.8225" y1="49.8475" x2="103.8225" y2="51.1175" width="0.4064" layer="1"/>
+<wire x1="103.8225" y1="51.1175" x2="106.045" y2="53.34" width="0.4064" layer="1"/>
+<wire x1="106.045" y1="53.34" x2="109.5375" y2="53.34" width="0.4064" layer="1"/>
+<wire x1="109.5375" y1="53.34" x2="110.1725" y2="52.705" width="0.4064" layer="1"/>
+<wire x1="110.1725" y1="52.705" x2="110.1725" y2="47.625" width="0.4064" layer="1"/>
+<wire x1="110.1725" y1="47.625" x2="109.5375" y2="46.99" width="0.4064" layer="1"/>
+<wire x1="109.5375" y1="46.99" x2="107.95" y2="46.99" width="0.4064" layer="1"/>
 </signal>
 <signal name="A6">
@@
 <wire x1="83.5025" y1="46.99" x2="86.995" y2="43.4975" width="0.4064" layer="1"/>
 <wire x1="86.995" y1="43.4975" x2="101.2825" y2="43.4975" width="0.4064" layer="1"/>
-<wire x1="101.2825" y1="43.4975" x2="103.8225" y2="46.0375" width="0.4064" layer="1"/>
-<wire x1="103.8225" y1="46.0375" x2="103.8225" y2="48.5775" width="0.4064" layer="1"/>
-<wire x1="103.8225" y1="48.5775" x2="104.775" y2="49.53" width="0.4064" layer="1"/>
-<wire x1="104.775" y1="49.53" x2="107.95" y2="49.53" width="0.4064" layer="1"/>
+<wire x1="101.2825" y1="43.4975" x2="107.315" y2="49.53" width="0.4064" layer="1"/>
+<wire x1="107.315" y1="49.53" x2="107.95" y2="49.53" width="0.4064" layer="1"/>
 </signal>
 <signal name="A7">
@@
 <wire x1="86.36" y1="46.0375" x2="87.9475" y2="44.45" width="0.4064" layer="1"/>
 <wire x1="87.9475" y1="44.45" x2="100.6475" y2="44.45" width="0.4064" layer="1"/>
-<wire x1="100.6475" y1="44.45" x2="102.87" y2="46.6725" width="0.4064" layer="1"/>
-<wire x1="102.87" y1="46.6725" x2="102.87" y2="50.8" width="0.4064" layer="1"/>
-<wire x1="102.87" y1="50.8" x2="104.14" y2="52.07" width="0.4064" layer="1"/>
-<wire x1="104.14" y1="52.07" x2="107.95" y2="52.07" width="0.4064" layer="1"/>
+<wire x1="100.6475" y1="44.45" x2="106.045" y2="49.8475" width="0.4064" layer="1"/>
+<wire x1="106.045" y1="49.8475" x2="106.045" y2="50.8" width="0.4064" layer="1"/>
+<wire x1="106.045" y1="50.8" x2="107.315" y2="52.07" width="0.4064" layer="1"/>
+<wire x1="107.315" y1="52.07" x2="108.585" y2="52.07" width="0.4064" layer="1"/>
+<wire x1="107.315" y1="52.07" x2="107.95" y2="52.07" width="0" layer="19" extent="1-1"/>
 </signal>
 <signal name="N$35">
@@
 <wire x1="52.125" y1="57.84" x2="52.705" y2="58.42" width="0.3048" layer="1"/>
 <via x="52.705" y="58.42" extent="1-16" drill="0.6" diameter="0.8128" shape="square"/>
-<wire x1="52.705" y1="58.42" x2="52.705" y2="43.18" width="0.3048" layer="16"/>
-<via x="52.705" y="43.18" extent="1-16" drill="0.6" diameter="0.8128" shape="square"/>
-<wire x1="52.705" y1="43.18" x2="55.88" y2="43.18" width="0.3048" layer="1"/>
+<wire x1="52.705" y1="58.42" x2="52.705" y2="45.085" width="0.3048" layer="16"/>
+<via x="52.705" y="45.085" extent="1-16" drill="0.6" diameter="0.8128" shape="square"/>
 <wire x1="55.88" y1="43.18" x2="58.42" y2="40.64" width="0.3048" layer="1"/>
+<wire x1="52.705" y1="45.085" x2="55.88" y2="43.18" width="0" layer="19" extent="1-1"/>
 </signal>
 <signal name="N$14">
