File: DoAnSpring2013/mmcaudio.brd (EAGLE design)
At the start: 181.9 x 121.9 mm, 84 parts, among them IC1 TL082, IC2 TL082, IC3 LM1117, IC4 TL082, IC5 TL082, U1 DAC0808LCN, U2 TEA2025B, X1 HD44780LCD-1602

Commit message: notthing to update
Parts:
- moved C27 33.8 mm to (156.8, 97.8)
- moved C28 33.8 mm to (174.0, 97.8)
- moved R5 33.8 mm to (57.5, 128.3)
- moved C14 33.8 mm to (92.7, 76.2)
- moved C24 33.8 mm to (163.8, 47.0)
- moved C25 33.8 mm to (152.4, 53.0)
- moved JP4 33.8 mm to (26.7, 33.0)
- moved LED1 33.8 mm to (27.9, 53.3)
- moved R16 33.8 mm to (76.2, 80.0)
- moved R18 33.8 mm to (68.6, 80.0)
- moved R21 33.8 mm to (72.4, 80.0)
- moved R23 33.8 mm to (138.7, 103.8)
- moved R30 33.8 mm to (177.8, 40.6)
- moved U2 33.8 mm to (156.2, 38.1)
- moved C11 33.8 mm to (45.7, 52.1)
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
Commit message: fsjdlfjsdlfjsdlfj
Parts:
- R16, R18, R20: value 6.8k -> 3.3k
- R17, R19, R21: value 6.8k -> 2.2k
- moved R21 6.35 mm to (66.0, 80.0)
- moved MMC/SD 3.81 mm to (44.5, 82.5), flipped to the bottom, turned to 0 degrees
- moved R18 2.54 mm to (71.1, 80.0)
- moved C13 1.27 mm to (55.9, 57.1), turned to 270 degrees
- moved IC3 1.27 mm to (45.7, 59.7), flipped to the bottom, turned to 270 degrees
Routing:
- net GND: track 1028.6 -> 752.3 mm, vias 9 -> 4
- net MISO: track 91.7 -> 0.00 mm
- net MOSI: track 53.4 -> 0.00 mm
- net N$38: track 35.2 -> 0.00 mm
- net CLK: track 25.4 -> 0.00 mm
- net N$40: track 24.8 -> 0.00 mm
- net CS: track 21.5 -> 0.00 mm
- net N$36: track 21.0 -> 0.00 mm
- net VCC: track 362.5 -> 352.1 mm, vias 0 -> 1
- net +3V3: track 50.6 -> 43.1 mm, vias 2 -> 0
- net -12V: track 520.8 -> 521.7 mm
- net N$30: track 56.0 -> 55.6 mm, vias 0 -> 3
- net +12V: vias 2 -> 0
- removed copper zone on layer 1, net GND
