File: DoAnSpring2013/mmcaudio.sch (EAGLE design)
At the start: 22 parts, among them IC1 TL082, IC2 TL082

Commit message: begin routing main board
Parts:
- added C10, C13: 222, datle-discrete:C-EUCERAMIC-CAP-COMMON
- added C11, C12, C15, C18, C7, C9: 100uF, datle-discrete:CPOL-USSANYO_D
- added C14, C21, C23, C24, C8: 223, datle-discrete:C-EUCERAMIC-CAP-COMMON
- added C16, C19, C22, C26, C30: 104, datle-discrete:C-EUCERAMIC-CAP-COMMON
- added C17: (no value), datle-discrete:CPOL-USSANYO_D
- added C20: 1uF, datle-discrete:CPOL-USSANYO_D
- added C25, C27, C28, C29: 10uF, datle-discrete:CPOL-USSANYO_D
- added IC3, IC4: TL082, datle-analogic:TL082
- added IC5: LM1117, datle-powerIC:V_REG_LM1117SOT223
- added IC6: (no value), datle-powerIC:V_REG_78XXSINK
- added JP4, JP5, JP9: (no value), datle-conn:PINHD-1X1
- added JP6: (no value), datle-conn:JP1E
- added JP8: SPEAKER, datle-conn:PINHD-1X20.5"
- added LED1: (no value), datle-discrete:LED5MM
- added Q1: (no value), datle-discrete:CRYSTALHC49S
- added R11, R23, R24, R25, R26, R27, R28: 6.8k, datle-discrete:R-US_0207/10
- added R12: 27k, datle-discrete:R-US_0207/10
- added R13, R14: 1.5k, datle-discrete:R-US_0207/10
- added R15: 10k, datle-discrete:R-TRIMM64W
- added R16, R17, R18, R19: 10k, datle-discrete:R-US_0207/10
- added R20, R30: 330, datle-discrete:R-US_0207/10
- added R21: 5k, datle-discrete:R-US_0207/10
- added R22, R29: 2k2, datle-discrete:R-US_0207/10
- added S1: (no value), datle-switch:10-XX
- added U$1: PIC18F4520-I/P, Microchip_By_element14_Batch_1:PIC18F4520-I/P
- added U1: TEA2025B, datle-analogic:TEA2025B
- added U2: DAC0808LCN, NSC_By_element14_Batch_1.1:DAC0808LCN
- added U3: SD_CARD_SOCKET4UCON, datle-discrete:SD_CARD_SOCKET4UCON
- added X1: HD44780LCD-1602, datle-display:HD44780LCD-1602
- C1, C6: device rcl:CPOL-USSANYO_A' -> datle-discrete:CPOL-USSANYO_D
- C2: value 222 -> 223; device rcl:C-EU025-060X050 -> datle-discrete:C-EUCERAMIC-CAP-COMMON
- C3: value 223 -> 222; device rcl:C-EU025-060X050 -> datle-discrete:C-EUCERAMIC-CAP-COMMON
- C4, C5: device rcl:C-EU025-060X050 -> datle-discrete:C-EUCERAMIC-CAP-COMMON
- JP1: device pinhead:PINHD-1X1 -> datle-conn:PINHD-1X6
- JP2: device pinhead:PINHD-1X1 -> datle-conn:PINHD-1X30.2"
- JP3: device pinhead:PINHD-1X4 -> datle-conn:PINHD-1X2
- R1: value 100k -> 1k; device rcl:R-TRIMM64W -> datle-discrete:R-US_0207/10
- R10, R2, R4, R5, R6, R7, R8, R9: device rcl:R-US_0207/10 -> datle-discrete:R-US_0207/10
- R3: value 1k -> 100k; device rcl:R-US_0207/10 -> datle-discrete:R-TRIMM64W
Connections:
- removed net N$12: D1.C, JP2.1, R10.1
- new net +3V3: C25.+, C26.1, IC5.OUT, U3.VDD
- new net A1-MSB: U$1.RD7/PSP7/P1D, U2.A1
- new net A2: U$1.RD6/PSP6/P1C, U2.A2
- new net A3: U$1.RD4/PSP4, U2.A3
- new net A4: U$1.RD3/PSP3, U2.A4
- new net A5: U$1.RD2/PSP2, U2.A5
- new net A6: U$1.RD1/PSP1, U2.A6
- new net A7: U$1.RD0/PSP0, U2.A7
- new net A8: U2.A8
- new net ADC: D1.C, JP5.1, R10.1, U$1.RA0/AN0
- new net B1: U$1.RB0/INT0/FLT0/AN12
- new net B2: U$1.RB1/INT1/AN10
- new net CLK: R24.1, R28.2, U$1.RC3/SCK/SCL
- new net CONTR: X1.VO
- new net CS: R23.2, R26.1, U$1.RC2/CCP1/P1A
- new net D4: U$1.RB2/INT2/AN8, X1.DB4
- new net D5: U$1.RB3/AN9/CCP2, X1.DB5
- new net D6: U$1.RB4/KBI0/AN11, X1.DB6
- new net D7: U$1.RB5/KBI1/PGM, X1.DB7
- new net E: U$1.RE1/~WR/AN6, X1.E
- new net IOUT: IC4B.OUT, R11.1, R29.1
- new net MISO: U$1.RC4/SDI/SDA, U3.DAT0
- new net MOSI: R25.1, R27.2, U$1.RC5/SDO
- new net N$13: C1.+, JP3.1, R17.1, R18.2
- new net N$14: C8.1, R11.2, R12.1
- new net N$15: C10.2, IC3A.+IN, R12.2
- new net N$16: C8.2, IC3A.-IN, IC3A.OUT, R13.1
- new net N$17: C14.1, R13.2, R14.2
- new net N$18: C13.2, IC3B.-IN, R14.1
- new net N$19: C14.2, C17.+, IC3B.+IN, IC3B.OUT
- new net N$20: C27.+, IC5.IN
- new net N$21: C17.-, JP9.1, R16.1
- new net N$22: C9.+, U1.FDBK_2
- new net N$23: C11.+, U1.FDBK
- new net N$24: C11.-, U1.BRIDGE
- new net N$25: C18.-, C19.2, JP8.1, U1.OUT.1
- new net N$26: C18.+, U1.BOOT.1
- new net N$27: C15.-, C16.2, U1.OUT.2
- new net N$28: C15.+, U1.BOOT.2
- new net N$29: C12.+, U1.SVR
- new net N$30: R15.E, R16.2
- new net N$31: C20.+, R2.1
- new net N$32: R20.1, X1.A
- new net N$33: C22.2, U2.COMP
- new net N$34: IC4B.-IN, R29.2, U2.IO
- new net N$35: U$1.RD5/PSP5/P1B
- new net N$36: R26.2, U3.CD/DAT3
- new net N$37: LED1.C, R30.2
- new net N$38: R25.2, U3.CMD
- new net N$40: R24.2, U3.CLK
- new net N$42: JP1.2, JP6.1
- new net OSC1: C23.2, Q1.1, U$1.OSC1/CLKI/RA7
- new net OSC2: C24.1, Q1.2, U$1.OSC2/CLKO/RA6
- new net PGC: JP1.5, U$1.RB6/KBI2/PGC
- new net PGD: JP1.4, U$1.RB7/KBI3/PGD
- new net PWR_AMP: R15.S, U1.IN.1(+)
- new net RESET: C21.1, JP1.1, R19.1, S1.S, S1.S1, U$1.~MCLR/VPP/RE3
- new net RS: U$1.RE0/~RD/AN5, X1.RS
- new net RX: U$1.RC7/RX/DT
- new net TX: U$1.RC6/TX/CK
- new net VDD: X1.VDD
- new net VREF+: R22.1, U2.VREF(+)
- new net VREF-: R21.2, U2.VREF(-)
- new net VSS: X1.DB0, X1.DB1, X1.DB2, X1.DB3, X1.RW, X1.VSS
- net +12V: now also C28.+, C7.+, IC3B.V-, IC4B.V-, IC6.IN, JP2.1, R17.2, U1.+VS; no longer JP3.3
- net -12V: now also C22.1, IC3B.V+, IC4B.V+, JP2.3, U2.VEE; no longer JP3.2
- net GND: now also C10.1, C12.-, C13.1, C16.1, C19.1, C20.-, C21.2, C23.1, C24.2, C25.-, C26.2, C27.-, C28.-, C29.-, C3.1, C30.2, C7.-, C9.-, IC4B.+IN, IC5.ADJ, IC6.GND, JP1.3, JP2.2, JP3.2, JP8.2, R1.1, R15.A, R18.1, R21.1, R23.1, R27.1, R28.1, R30.1, S1.P, S1.P1, U$1.VSS, U1.GND, U1.GND(SUB), U1.GND_2, U1.GND_3, U1.GND_4, U1.IN.2(+), U2.GND, U3.VSS1, U3.VSS2, X1.K; no longer C2.1, JP3.1, R2.1, R3.1
- net N$1: now also R1.2; no longer R2.2
- net N$2: now also R2.2, R3.A; no longer R1.A, R3.2
- net N$3: now also JP4.1, R3.S; no longer JP1.1, R1.S
- net N$4: now also C2.1; no longer C3.1
- net N$5: now also C3.2; no longer C2.2
- net N$6: now also C2.2; no longer C3.2
- net VCC: now also C29.+, C30.1, IC6.OUT, JP6.2, LED1.A, R19.2, R20.2, R22.2, U$1.VDD, U$1.VDD_2, U2.VCC; no longer JP3.4
Other:
- moved on the sheet: C2, C3, C4, D1, R2, R9

Commit message: routing
Parts:
- removed IC6: (no value), datle-powerIC:V_REG_78XXSINK
- removed JP9: (no value), datle-conn:PINHD-1X1
- removed R3: 100k, datle-discrete:R-TRIMM64W
- removed U3: SD_CARD_SOCKET4UCON, datle-discrete:SD_CARD_SOCKET4UCON
- added JP7: SPEAKER, datle-conn:PINHD-1X20.5"
- added LM1: (no value), datle-powerIC:V_REG_78XXSINK
- added MMC/SD: SD_CARD_SOCKET4UCON, datle-discrete:SD_CARD_SOCKET4UCON
- added R31: 10k, datle-discrete:R-TRIMM
- C10: value 222 -> 104
- C11: value 100uF -> 104; device datle-discrete:CPOL-USSANYO_D -> datle-discrete:C-EUCERAMIC-CAP-COMMON
- C12, C7, C9: value 100uF -> 10uF
- C13: value 222 -> 10uF; device datle-discrete:C-EUCERAMIC-CAP-COMMON -> datle-discrete:CPOL-USSANYO_D
- C15: value 100uF -> 223; device datle-discrete:CPOL-USSANYO_D -> datle-discrete:C-EUCERAMIC-CAP-COMMON
- C16, C26: value 104 -> 223
- C17: value (none) -> 104; device datle-discrete:CPOL-USSANYO_D -> datle-discrete:C-EUCERAMIC-CAP-COMMON
- C19, C22: value 104 -> 100uF; device datle-discrete:C-EUCERAMIC-CAP-COMMON -> datle-discrete:CPOL-USSANYO_D
- C2: value 223 -> 1uF; device datle-discrete:C-EUCERAMIC-CAP-COMMON -> datle-discrete:CPOL-USSANYO_D
- C20: value 1uF -> 100uF
- C21, C24: value 223 -> 100uF; device datle-discrete:C-EUCERAMIC-CAP-COMMON -> datle-discrete:CPOL-USSANYO_D
- C23: value 223 -> 104
- C25: value 10uF -> 104; device datle-discrete:CPOL-USSANYO_D -> datle-discrete:C-EUCERAMIC-CAP-COMMON
- C27, C28: value 10uF -> 222; device datle-discrete:CPOL-USSANYO_D -> datle-discrete:C-EUCERAMIC-CAP-COMMON
- C29, C6: value 10uF -> 223; device datle-discrete:CPOL-USSANYO_D -> datle-discrete:C-EUCERAMIC-CAP-COMMON
- C3: value 222 -> 223
- C30: value 104 -> (none); device datle-discrete:C-EUCERAMIC-CAP-COMMON -> datle-discrete:CPOL-USSANYO_D
- C4: value 103 -> 222
- C5: value 223 -> 103
- C8: value 223 -> 10uF; device datle-discrete:C-EUCERAMIC-CAP-COMMON -> datle-discrete:CPOL-USSANYO_D
- IC3: value TL082 -> LM1117; device datle-analogic:TL082 -> datle-powerIC:V_REG_LM1117SOT223
- IC5: value LM1117 -> TL082; device datle-powerIC:V_REG_LM1117SOT223 -> datle-analogic:TL082
- JP1: device datle-conn:PINHD-1X6 -> datle-conn:PINHD-1X2
- JP2: device datle-conn:PINHD-1X30.2" -> datle-conn:PINHD-1X1
- JP3: device datle-conn:PINHD-1X2 -> datle-conn:PINHD-1X1
- JP4: device datle-conn:PINHD-1X1 -> datle-conn:PINHD-1X30.2"
- JP5: device datle-conn:PINHD-1X1 -> datle-conn:PINHD-1X6
- JP8: value SPEAKER -> (none); device datle-conn:PINHD-1X20.5" -> datle-conn:PINHD-1X1
- R1, R10, R2: value 1k -> 10k
- R11: value 6.8k -> 10k
- R12: value 27k -> 1k
- R13: value 1.5k -> 330
- R14: value 1.5k -> 10k
- R15: value 10k -> 330; device datle-discrete:R-TRIMM64W -> datle-discrete:R-US_0207/10
- R16: value 10k -> 100
- R17, R18, R19: value 10k -> 6.8k
- R20: value 330 -> 6.8k
- R21: value 5k -> 6.8k
- R22: value 2k2 -> 6.8k
- R23, R25: value 6.8k -> 2k2
- R24: value 6.8k -> 5k
- R27: value 6.8k -> 27k
- R28: value 6.8k -> 1.5k
- R29: value 2k2 -> 1.5k
- R30: value 330 -> 10k
- R4: value 6.8k -> 1k
- R5: value 27k -> 100k; device datle-discrete:R-US_0207/10 -> datle-discrete:R-TRIMM64W
- R6: value 3.3k -> 6.8k
- R7: value 3.3k -> 27k
- R8, R9: value 10k -> 3.3k
- U$1: device Microchip_By_element14_Batch_1:PIC18F4520-I/P -> datle-mcu:PIC18F4520-I/P
- U1: value TEA2025B -> DAC0808LCN; device datle-analogic:TEA2025B -> datle-analogic:DAC0808LCN
- U2: value DAC0808LCN -> TEA2025B; device NSC_By_element14_Batch_1.1:DAC0808LCN -> datle-analogic:TEA2025B
Connections:
- removed net N$20: C27.+, IC5.IN
- net +12V: now also C18.+, C8.+, IC5B.V-, JP4.1, LM1.IN, R1.2, U2.+VS; no longer C28.+, C7.+, IC3B.V-, IC6.IN, JP2.1, R17.2, U1.+VS
- net +3V3: now also C11.1, C12.+, IC3.OUT, MMC/SD.VDD; no longer C25.+, C26.1, IC5.OUT, U3.VDD
- net -12V: now also C17.2, IC5B.V+, JP4.3, U1.VEE; no longer C22.1, IC3B.V+, JP2.3, U2.VEE
- net A1-MSB: now also U1.A1; no longer U2.A1
- net A2: now also U1.A2; no longer U2.A2
- net A3: now also U1.A3; no longer U2.A3
- net A4: now also U1.A4; no longer U2.A4
- net A5: now also U1.A5; no longer U2.A5
- net A6: now also U1.A6; no longer U2.A6
- net A7: now also U1.A7; no longer U2.A7
- net A8: now also U1.A8; no longer U2.A8
- net ADC: now also JP3.1, R12.1; no longer JP5.1, R10.1
- net CLK: now also R21.2, R22.1; no longer R24.1, R28.2
- net CONTR: now also R15.1
- net CS: now also R17.2, R18.1; no longer R23.2, R26.1
- net GND: now also C10.2, C11.2, C13.-, C14.1, C15.2, C16.2, C18.-, C19.-, C2.-, C21.-, C25.1, C27.1, C28.1, C5.1, C8.-, IC3.ADJ, JP1.2, JP4.2, JP5.3, JP7.2, LM1.GND, MMC/SD.VSS1, MMC/SD.VSS2, R11.2, R13.1, R17.1, R19.1, R2.1, R24.1, R31.A, U$1.VSS_2, U2.GND(SUB), U2.GND_2, U2.GND_3, U2.GND_4, U2.IN.2(+); no longer C10.1, C13.1, C16.1, C19.1, C20.-, C21.2, C24.2, C25.-, C26.2, C27.-, C28.-, C29.-, C3.1, C30.2, C7.-, IC5.ADJ, IC6.GND, JP1.3, JP2.2, JP3.2, JP8.2, R1.1, R15.A, R18.1, R23.1, R27.1, R28.1, R30.1, R9.2, U1.GND(SUB), U1.GND_2, U1.GND_3, U1.GND_4, U1.IN.2(+), U3.VSS1, U3.VSS2
- net IOUT: now also R25.1, R26.1; no longer R11.1, R29.1
- net MISO: now also MMC/SD.DAT0; no longer U3.DAT0
- net MOSI: now also R19.2, R20.1; no longer R25.1, R27.2
- net N$1: no longer R1.2
- net N$10: now also C7.+, R10.1, R11.1; no longer C6.+, R8.1, R9.1
- net N$11: now also R12.2; no longer R10.2
- net N$13: now also JP1.1, R1.1, R2.2; no longer JP3.1, R17.1, R18.2
- net N$14: now also C26.1, R26.2, R27.1; no longer C8.1, R11.2, R12.1
- net N$15: now also C27.2, IC5A.+IN, R27.2; no longer C10.2, IC3A.+IN, R12.2
- net N$16: now also C26.2, IC5A.-IN, IC5A.OUT, R28.1; no longer C8.2, IC3A.-IN, IC3A.OUT, R13.1
- net N$17: now also C29.1, R28.2, R29.2; no longer C14.1, R13.2, R14.2
- net N$18: now also C28.2, IC5B.-IN, R29.1; no longer C13.2, IC3B.-IN, R14.1
- net N$19: now also C29.2, C30.+, IC5B.+IN, IC5B.OUT; no longer C14.2, C17.+, IC3B.+IN, IC3B.OUT
- net N$2: now also R4.2, R5.A; no longer R2.2, R3.A
- net N$21: now also C30.-, JP8.1, R30.1; no longer C17.-, JP9.1, R16.1
- net N$22: now also C19.+, U2.FDBK_2; no longer C9.+, U1.FDBK_2
- net N$23: now also C20.+, U2.FDBK; no longer C11.+, U1.FDBK
- net N$24: now also C20.-, U2.BRIDGE; no longer C11.-, U1.BRIDGE
- net N$25: now also C24.-, C25.2, JP7.1, U2.OUT.1; no longer C18.-, C19.2, JP8.1, U1.OUT.1
- net N$26: now also C24.+, U2.BOOT.1; no longer C18.+, U1.BOOT.1
- net N$27: now also C22.-, C23.2, U2.OUT.2; no longer C15.-, C16.2, U1.OUT.2
- net N$28: now also C22.+, U2.BOOT.2; no longer C15.+, U1.BOOT.2
- net N$29: now also C21.+, U2.SVR; no longer C12.+, U1.SVR
- net N$3: now also JP2.1, R5.S, R6.1; no longer JP4.1, R3.S, R4.1
- net N$30: now also R30.2, R31.E; no longer R15.E, R16.2
- net N$31: now also C2.+, R4.1; no longer C20.+, R2.1
- net N$32: now also R16.1; no longer R20.1
- net N$33: now also C17.1, U1.COMP; no longer C22.2, U2.COMP
- net N$34: now also R25.2, U1.IO; no longer R29.2, U2.IO
- net N$36: now also MMC/SD.CD/DAT3, R18.2; no longer R26.2, U3.CD/DAT3
- net N$37: now also R13.2; no longer R30.2
- net N$38: now also MMC/SD.CMD, R20.2; no longer R25.2, U3.CMD
- net N$4: now also C3.1, R6.2, R7.1; no longer C2.1, R4.2, R5.1
- net N$40: now also MMC/SD.CLK, R22.2; no longer R24.2, U3.CLK
- net N$42: now also JP5.2; no longer JP1.2
- net N$5: now also C4.2, R7.2; no longer C3.2, R5.2
- net N$6: now also C3.2, R8.1; no longer C2.2, R6.1
- net N$7: now also C6.1, R8.2, R9.2; no longer C5.1, R6.2, R7.2
- net N$8: now also C5.2, R9.1; no longer C4.2, R7.1
- net N$9: now also C6.2, C7.-; no longer C5.2, C6.-
- net OSC1: now also C14.2; no longer C23.2
- net OSC2: now also C15.1; no longer C24.1
- net PGC: now also JP5.5; no longer JP1.5
- net PGD: now also JP5.4; no longer JP1.4
- net PWR_AMP: now also R31.S, U2.IN.1(+); no longer R15.S, U1.IN.1(+)
- net RESET: now also C16.1, JP5.1, R14.1; no longer C21.1, JP1.1, R19.1
- net VCC: now also C10.1, C13.+, C9.+, IC3.IN, LM1.OUT, R10.2, R14.2, R16.2, R23.2, U1.VCC; no longer C29.+, C30.1, IC6.OUT, R19.2, R20.2, R22.2, R8.2, U2.VCC
- net VDD: now also R15.2
- net VREF+: now also R23.1, U1.VREF(+); no longer R22.1, U2.VREF(+)
- net VREF-: now also R24.2, U1.VREF(-); no longer R21.2, U2.VREF(-)
Other:
- note added: "DAC"
- note added: "Display"
- note added: "MMC Supply"
- note added: "MMC/SD"
- note added: "Main controller"
- note added: "Main supply"
- note added: "Mic Input"
- note added: "Power amp"
- note added: "Reconstruction"

Commit message: add button B1 & B2
Parts:
- removed R31: 10k, datle-discrete:R-TRIMM
- added R3: 1k, datle-discrete:R-US_0207/10
- added S2, S3: (no value), datle-switch:10-XX
- C14, C15: value 223 -> 22p
- C16: value 223 -> 104
- R11: value 10k -> 1k
- R12: value 1k -> 330
- R13: value 330 -> 10k
- R14: value 10k -> 330
- R15: value 330 -> 100
- R16: value 100 -> 6.8k
- R22: value 6.8k -> 2k2
- R23: value 2k2 -> 5k
- R24: value 5k -> 2k2
- R25: value 2k2 -> 6.8k
- R26, R6: value 6.8k -> 27k
- R27: value 27k -> 1.5k
- R29: value 1.5k -> 10k
- R30: device datle-discrete:R-US_0207/10 -> datle-discrete:R-TRIMM
- R4: value 1k -> 100k; device datle-discrete:R-US_0207/10 -> datle-discrete:R-TRIMM64W
- R5: value 100k -> 6.8k; device datle-discrete:R-TRIMM64W -> datle-discrete:R-US_0207/10
- R7: value 27k -> 3.3k
- R9: value 3.3k -> 10k
Connections:
- net ADC: now also R11.1; no longer R12.1
- net B1: now also S1.S, S1.S1
- net B2: now also S2.S, S2.S1
- net CLK: now also R20.2, R21.1; no longer R21.2, R22.1
- net CONTR: now also R14.1; no longer R15.1
- net CS: now also R16.2, R17.1; no longer R17.2, R18.1
- net GND: now also R10.2, R12.1, R16.1, R18.1, R20.1, R23.1, R30.A, S2.P, S2.P1, S3.P, S3.P1; no longer R11.2, R13.1, R17.1, R19.1, R21.1, R24.1, R31.A
- net IOUT: now also R24.1; no longer R26.1
- net MOSI: now also R18.2, R19.1; no longer R19.2, R20.1
- net N$10: now also R9.1; no longer R11.1
- net N$11: now also R11.2; no longer R12.2
- net N$14: now also R25.2, R26.1; no longer R26.2, R27.1
- net N$15: now also R26.2; no longer R27.2
- net N$16: now also R27.1; no longer R28.1
- net N$17: now also R27.2; no longer R29.2
- net N$18: now also R28.1; no longer R29.1
- net N$2: now also R3.2, R4.A; no longer R4.2, R5.A
- net N$21: now also R29.1; no longer R30.1
- net N$3: now also R4.S, R5.1; no longer R5.S, R6.1
- net N$30: now also R29.2, R30.E; no longer R30.2, R31.E
- net N$31: now also R3.1; no longer R4.1
- net N$32: now also R15.1; no longer R16.1
- net N$34: now also R24.2; no longer R25.2
- net N$36: now also R17.2; no longer R18.2
- net N$37: now also R12.2; no longer R13.2
- net N$38: now also R19.2; no longer R20.2
- net N$4: now also R5.2, R6.1; no longer R6.2, R7.1
- net N$40: now also R21.2; no longer R22.2
- net N$5: now also R6.2; no longer R7.2
- net N$6: now also R7.1; no longer R8.1
- net N$7: now also R7.2; no longer R9.2
- net N$8: now also R8.1; no longer R9.1
- net PWR_AMP: now also R30.S; no longer R31.S
- net RESET: now also R13.1, S3.S, S3.S1; no longer R14.1, S1.S, S1.S1
- net VCC: now also R13.2, R15.2, R22.2, R9.2; no longer R10.2, R14.2, R16.2, R23.2
- net VDD: now also R14.2; no longer R15.2
- net VREF+: now also R22.1; no longer R23.1
- net VREF-: now also R23.2; no longer R24.2
Other:
- moved on the sheet: C14, C15, JP5, JP6, Q1, R10, R11, R12, R14, R15, R16, R17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

Commit message: routing failed 12:56SA 20131105
Parts:
- removed JP7: SPEAKER, datle-conn:PINHD-1X20.5"
- removed JP8: (no value), datle-conn:PINHD-1X1
- JP5: value (none) -> SPEAKER; device datle-conn:PINHD-1X6 -> datle-conn:PINHD-1X20.5"
- JP6: device datle-conn:JP1E -> datle-conn:PINHD-1X1
- R14: value 330 -> 4k7
Connections:
- removed net N$42: JP5.2, JP6.1
- net D4: now also U$1.RB5/KBI1/PGM; no longer U$1.RB2/INT2/AN8
- net D5: now also U$1.RB4/KBI0/AN11; no longer U$1.RB3/AN9/CCP2
- net D6: now also U$1.RB3/AN9/CCP2; no longer U$1.RB4/KBI0/AN11
- net D7: now also U$1.RB2/INT2/AN8; no longer U$1.RB5/KBI1/PGM
- net GND: now also JP5.2; no longer JP5.3, JP7.2
- net N$21: now also JP6.1; no longer JP8.1
- net N$25: now also JP5.1; no longer JP7.1
- net PGC: no longer JP5.5
- net PGD: no longer JP5.4
- net RESET: no longer JP5.1
- net VCC: no longer JP6.2
Other:
- moved on the sheet: R23

Commit message: route done 1
Parts:
- added JP7: (no value), datle-conn:PINHD-1X1
Connections:
- removed net N$35: U$1.RD5/PSP5/P1B
- removed net PGC: U$1.RB6/KBI2/PGC
- removed net PGD: U$1.RB7/KBI3/PGD
- net A3: now also U$1.RD5/PSP5/P1B; no longer U$1.RD4/PSP4
- net A4: now also U$1.RD4/PSP4; no longer U$1.RD3/PSP3
- net A5: now also U$1.RD3/PSP3; no longer U$1.RD2/PSP2
- net A6: now also U$1.RD2/PSP2; no longer U$1.RD1/PSP1
- net A7: now also U$1.RD1/PSP1; no longer U$1.RD0/PSP0
- net A8: now also U$1.RD0/PSP0
- net E: now also U$1.RB6/KBI2/PGC; no longer U$1.RE1/~WR/AN6
- net RS: now also U$1.RB7/KBI3/PGD; no longer U$1.RE0/~RD/AN5
- net TX: now also JP7.1
Changed lines of the file:
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@@
 <setting verticaltext="up"/>
 </settings>
-<grid distance="0.1" unitdist="inch" unit="inch" style="lines" multiple="1" display="no" altdistance="0.01" altunitdist="inch" altunit="mil"/>
+<grid distance="50" unitdist="mil" unit="mil" style="lines" multiple="1" display="yes" altdistance="0.01" altunitdist="inch" altunit="mil"/>
 <layers>
 <layer number="1" name="Top" color="4" fill="1" visible="no" active="no"/>
@@
 <part name="GND1" library="supply1" deviceset="GND" device=""/>
 <part name="GND19" library="supply1" deviceset="GND" device=""/>
+<part name="JP7" library="datle-conn" deviceset="PINHD-1X1" device=""/>
 </parts>
 <sheets>
@@
 <instance part="GND1" gate="1" x="66.04" y="99.06"/>
 <instance part="GND19" gate="1" x="81.28" y="99.06"/>
+<instance part="JP7" gate="G$1" x="63.5" y="163.83" rot="R180"/>
 </instances>
 <busses>
@@
 </segment>
 <segment>
-<pinref part="U$1" gate="A" pin="RE0/~RD/AN5"/>
-<wire x1="243.84" y1="119.38" x2="255.27" y2="119.38" width="0.1524" layer="91"/>
-<label x="246.38" y="119.38" size="1.778" layer="95"/>
+<pinref part="U$1" gate="A" pin="RB7/KBI3/PGD"/>
+<wire x1="243.84" y1="147.32" x2="255.27" y2="147.32" width="0.1524" layer="91"/>
+<label x="246.38" y="147.32" size="1.778" layer="95"/>
 </segment>
 </net>
@@
 <label x="316.23" y="138.43" size="1.778" layer="95" rot="R90"/>
 </segment>
-<segment>
-<pinref part="U$1" gate="A" pin="RE1/~WR/AN6"/>
-<wire x1="243.84" y1="116.84" x2="255.27" y2="116.84" width="0.1524" layer="91"/>
-<label x="246.38" y="116.84" size="1.778" layer="95"/>
-</segment>
-</net>
-<net name="PGD" class="0">
-<segment>
-<pinref part="U$1" gate="A" pin="RB7/KBI3/PGD"/>
-<wire x1="243.84" y1="147.32" x2="255.27" y2="147.32" width="0.1524" layer="91"/>
-<label x="246.38" y="147.32" size="1.778" layer="95"/>
-</segment>
-</net>
-<net name="PGC" class="0">
 <segment>
 <pinref part="U$1" gate="A" pin="RB6/KBI2/PGC"/>
@@
 <label x="246.38" y="127" size="1.778" layer="95"/>
 </segment>
+<segment>
+<pinref part="JP7" gate="G$1" pin="1"/>
+<wire x1="66.04" y1="163.83" x2="85.09" y2="163.83" width="0.1524" layer="91"/>
+<label x="74.93" y="163.83" size="1.778" layer="95"/>
+</segment>
 </net>
 <net name="RX" class="0">
@@
 </segment>
 </net>
-<net name="A3" class="0">
+<net name="A4" class="0">
 <segment>
 <pinref part="U$1" gate="A" pin="RD4/PSP4"/>
-<wire x1="129.54" y1="119.38" x2="142.24" y2="119.38" width="0.1524" layer="91"/>
-<label x="132.08" y="116.84" size="1.778" layer="95"/>
+<wire x1="142.24" y1="119.38" x2="129.54" y2="119.38" width="0.1524" layer="91"/>
 <label x="132.08" y="119.38" size="1.778" layer="95"/>
 </segment>
 </net>
-<net name="A4" class="0">
+<net name="A5" class="0">
 <segment>
 <pinref part="U$1" gate="A" pin="RD3/PSP3"/>
@@
 </segment>
 </net>
-<net name="A5" class="0">
+<net name="A6" class="0">
 <segment>
 <pinref part="U$1" gate="A" pin="RD2/PSP2"/>
@@
 </segment>
 </net>
-<net name="A6" class="0">
+<net name="A7" class="0">
 <segment>
 <pinref part="U$1" gate="A" pin="RD1/PSP1"/>
@@
 </segment>
 </net>
-<net name="A7" class="0">
-<segment>
-<pinref part="U$1" gate="A" pin="RD0/PSP0"/>
-<wire x1="142.24" y1="129.54" x2="129.54" y2="129.54" width="0.1524" layer="91"/>
-<label x="132.08" y="129.54" size="1.778" layer="95"/>
-</segment>
-</net>
-<net name="N$35" class="0">
+<net name="A3" class="0">
 <segment>
 <pinref part="U$1" gate="A" pin="RD5/PSP5/P1B"/>
 <wire x1="142.24" y1="116.84" x2="129.54" y2="116.84" width="0.1524" layer="91"/>
+<label x="132.08" y="116.84" size="1.778" layer="95"/>
 </segment>
 </net>
@@
 </segment>
 </net>
+<net name="A8" class="0">
+<segment>
+<pinref part="U$1" gate="A" pin="RD0/PSP0"/>
+<wire x1="142.24" y1="129.54" x2="129.54" y2="129.54" width="0.1524" layer="91"/>
+<label x="132.08" y="129.54" size="1.778" layer="95"/>
+</segment>
+</net>

Commit message: clean the fault
Parts:
- R16, R18, R20: value 6.8k -> 3.3k
- R17, R19, R21: value 6.8k -> 2.2k
Changed lines of the file:
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@@
 <setting verticaltext="up"/>
 </settings>
-<grid distance="50" unitdist="mil" unit="mil" style="lines" multiple="1" display="yes" altdistance="0.01" altunitdist="inch" altunit="mil"/>
+<grid distance="0.1" unitdist="inch" unit="inch" style="lines" multiple="1" display="no" altdistance="0.01" altunitdist="inch" altunit="inch"/>
 <layers>
 <layer number="1" name="Top" color="4" fill="1" visible="no" active="no"/>
@@
 <part name="MMC/SD" library="datle-discrete" deviceset="SD_CARD_SOCKET" device="4UCON"/>
 <part name="GND28" library="supply1" deviceset="GND" device=""/>
-<part name="R21" library="datle-discrete" deviceset="R-US_" device="0207/10" value="6.8k"/>
-<part name="R19" library="datle-discrete" deviceset="R-US_" device="0207/10" value="6.8k"/>
-<part name="R17" library="datle-discrete" deviceset="R-US_" device="0207/10" value="6.8k"/>
-<part name="R16" library="datle-discrete" deviceset="R-US_" device="0207/10" value="6.8k"/>
-<part name="R18" library="datle-discrete" deviceset="R-US_" device="0207/10" value="6.8k"/>
-<part name="R20" library="datle-discrete" deviceset="R-US_" device="0207/10" value="6.8k"/>
+<part name="R21" library="datle-discrete" deviceset="R-US_" device="0207/10" value="2.2k"/>
+<part name="R19" library="datle-discrete" deviceset="R-US_" device="0207/10" value="2.2k"/>
+<part name="R17" library="datle-discrete" deviceset="R-US_" device="0207/10" value="2.2k"/>
+<part name="R16" library="datle-discrete" deviceset="R-US_" device="0207/10" value="3.3k"/>
+<part name="R18" library="datle-discrete" deviceset="R-US_" device="0207/10" value="3.3k"/>
+<part name="R20" library="datle-discrete" deviceset="R-US_" device="0207/10" value="3.3k"/>
 <part name="GND29" library="supply1" deviceset="GND" device=""/>
 <part name="GND30" library="supply1" deviceset="GND" device=""/>
